Commit message: Updated URDF

File: urdf/artus_lite_mk7/left_hand/robot.urdf (robot description, URDF)
Before this commit: robot ArtusLite_LeftHand, 22 links, 21 joints
Links:
- removed link l_d1-1_urdf
- removed link l_d1-2_urdf
- removed link l_d1-3_urdf
- removed link l_d1-4_urdf
- removed link l_d2-1_urdf
- removed link l_d2-2_urdf
- removed link l_d2-3_urdf
- removed link l_d2-4_urdf
- removed link l_d3-1_urdf
- removed link l_d3-2_urdf
- removed link l_d3-3_urdf
- removed link l_d3-4_urdf
- removed link l_d4-1_urdf
- removed link l_d4-2_urdf
- removed link l_d4-3_urdf
- removed link l_d4-4_urdf
- removed link l_t1_urdf
- removed link l_t2_urdf
- removed link l_t3_urdf
- removed link l_t4_urdf
- added link d1-1_urdf, mass 0.0096628566425330745387; collision mesh filename=meshes/d1-1_urdf.stl; visual mesh filename=meshes/d1-1_urdf.stl
- added link d1-2_urdf, mass 0.009662856642533072804; collision mesh filename=meshes/d1-2_urdf.stl; visual mesh filename=meshes/d1-2_urdf.stl
- added link d1-3_urdf, mass 0.0096628566425330745387; collision mesh filename=meshes/d1-3_urdf.stl; visual mesh filename=meshes/d1-3_urdf.stl
- added link d1-4_urdf, mass 0.009662856642533072804; collision mesh filename=meshes/d1-4_urdf.stl; visual mesh filename=meshes/d1-4_urdf.stl
- added link d2-1_urdf, mass 0.011864989574403397507; collision mesh filename=meshes/d2-1_urdf.stl; visual mesh filename=meshes/d2-1_urdf.stl
- added link d2-2_urdf, mass 0.011864989574403399242; collision mesh filename=meshes/d2-2_urdf.stl; visual mesh filename=meshes/d2-2_urdf.stl
- added link d2-3_urdf, mass 0.011864989574403397507; collision mesh filename=meshes/d2-3_urdf.stl; visual mesh filename=meshes/d2-3_urdf.stl
- added link d2-4_urdf, mass 0.011864989574403399242; collision mesh filename=meshes/d2-4_urdf.stl; visual mesh filename=meshes/d2-4_urdf.stl
- added link d3-1_urdf, mass 0.022614819883081289931; collision mesh filename=meshes/d3-1_urdf.stl; visual mesh filename=meshes/d3-1_urdf.stl
- added link d3-2_urdf, mass 0.0226148198830812934; collision mesh filename=meshes/d3-2_urdf.stl; visual mesh filename=meshes/d3-2_urdf.stl
- added link d3-3_urdf, mass 0.022614819883081289931; collision mesh filename=meshes/d3-3_urdf.stl; visual mesh filename=meshes/d3-3_urdf.stl
- added link d3-4_urdf, mass 0.022614819883081289931; collision mesh filename=meshes/d3-4_urdf.stl; visual mesh filename=meshes/d3-4_urdf.stl
- added link d4-1_urdf, mass 0.007132231448786834245; collision mesh filename=meshes/d4-1_urdf.stl; visual mesh filename=meshes/d4-1_urdf.stl
- added link d4-2_urdf, mass 0.007132231448786834245; collision mesh filename=meshes/d4-2_urdf.stl; visual mesh filename=meshes/d4-2_urdf.stl
- added link d4-3_urdf, mass 0.0071322314487868333777; collision mesh filename=meshes/d4-3_urdf.stl; visual mesh filename=meshes/d4-3_urdf.stl
- added link d4-4_urdf, mass 0.007132231448786834245; collision mesh filename=meshes/d4-4_urdf.stl; visual mesh filename=meshes/d4-4_urdf.stl
- added link t1_urdf, mass 0.011648615104362203959; collision mesh filename=meshes/t1_urdf.stl; visual mesh filename=meshes/t1_urdf.stl
- added link t2_urdf, mass 0.014650153995995375544; collision mesh filename=meshes/t2_urdf.stl; visual mesh filename=meshes/t2_urdf.stl
- added link t3_urdf, mass 0.030585609045160683933; collision mesh filename=meshes/t3_urdf.stl; visual mesh filename=meshes/t3_urdf.stl
- added link t4_urdf, mass 0.010288104754589431911; collision mesh filename=meshes/t4_urdf.stl; visual mesh filename=meshes/t4_urdf.stl
- link left_forearm_and_palm_assembly: mass 0.35338696093763821704 -> 0.68622918239401642371
Joints:
- removed joint l_index_01
- removed joint l_index_12
- removed joint l_index_23
- removed joint l_index_34
- removed joint l_middle_01
- removed joint l_middle_12
- removed joint l_middle_23
- removed joint l_middle_34
- removed joint l_pinky_01
- removed joint l_pinky_12
- removed joint l_pinky_23
- removed joint l_pinky_34
- removed joint l_ring_01
- removed joint l_ring_12
- removed joint l_ring_23
- removed joint l_ring_34
- removed joint l_thumb_01
- removed joint l_thumb_12
- removed joint l_thumb_23
- removed joint l_thumb_34
- added joint index_01: type revolute, parent left_forearm_and_palm_assembly, child d4-4_urdf, origin xyz=0.0352612563274789792 0.19513802398559310092 -0.010513965579231661016 rpy=3.0543261909900740747 -2.6020852139652102472e-15 -1.6100662349647958393, axis 0 0 1, limit lower=-0.29670597283903604735 upper=0.29670597283903604735 effort=1 velocity=20
- added joint index_12: type revolute, parent d4-4_urdf, child d3-4_urdf, origin xyz=-0.015274999999999872013 0.0072500000000000966449 -0.0077499999999998967284 rpy=-1.5707963267948976682 -1.5707963267948830133 0, axis 0 0 1, limit lower=-0.034906585039886590949 upper=1.570796326794896558 effort=1 velocity=20
- added joint index_23: type revolute, parent d3-4_urdf, child d2-4_urdf, origin xyz=-0.0010000000000000412205 -0.037874999999999964251 -0.00050000000000011840529 rpy=-2.4817590593525338253e-15 2.570777650635345777e-15 -1.5707963267948958919, axis 0 0 1, limit lower=0 upper=1.570796326794896558 effort=1 velocity=20
- added joint index_34: type revolute, parent d2-4_urdf, child d1-4_urdf, origin xyz=0.026000000000000050848 -5.0957502106818708398e-18 -0.00049999999999996574962 rpy=1.4027645268064363647e-15 -2.2530004780047258679e-15 -1.57079632679489678, axis 0 0 1, limit lower=0 upper=1.570796326794896558 effort=1 velocity=20
- added joint middle_01: type revolute, parent left_forearm_and_palm_assembly, child d4-3_urdf, origin xyz=0.011738453089343185015 0.19915000000000054881 -0.0080006470225532679008 rpy=3.1415926535897926719 1.307825854535432319e-16 -1.57079632679489678, axis 0 0 1, limit lower=-0.29670597283903604735 upper=0.29670597283903604735 effort=1 velocity=20
- added joint middle_12: type revolute, parent d4-3_urdf, child d3-3_urdf, origin xyz=-0.015275000000000010791 0.0072500000000000402664 -0.0077499999999999453007 rpy=-1.57079632679489678 -1.5707963267948961139 0, axis 0 0 1, limit lower=-0.034906585039886590949 upper=1.570796326794896558 effort=1 velocity=20
- added joint middle_23: type revolute, parent d3-3_urdf, child d2-3_urdf, origin xyz=-0.001000000000000215777 -0.037874999999999825473 -0.00050000000000005248579 rpy=-1.0155656137714762e-15 -8.1269680571163029421e-16 -1.5707963267948970021, axis 0 0 1, limit lower=0 upper=1.570796326794896558 effort=1 velocity=20
- added joint middle_34: type revolute, parent d2-3_urdf, child d1-3_urdf, origin xyz=0.026000000000000134115 -4.5536491244391186228e-18 -0.00050000000000000044409 rpy=-2.9646186017117878309e-15 3.6635847905925687338e-16 -1.5707963267948532593, axis 0 0 1, limit lower=0 upper=1.570796326794896558 effort=1 velocity=20
- added joint pinky_01: type revolute, parent left_forearm_and_palm_assembly, child d4-1_urdf, origin xyz=-0.035163940960675876823 0.18909438839224840256 -0.014053824767915700997 rpy=-2.9670597283903603625 -1.5269348559829246889e-15 -1.4791665410651910761, axis 0 0 1, limit lower=-0.29670597283903604735 upper=0.29670597283903604735 effort=1 velocity=20
- added joint pinky_12: type revolute, parent d4-1_urdf, child d3-1_urdf, origin xyz=-0.015275000000000038547 0.0072500000000000792977 -0.0077499999999998108596 rpy=-1.5707963267948972241 -1.5707963267948952257 0, axis 0 0 1, limit lower=-0.034906585039886590949 upper=1.570796326794896558 effort=1 velocity=20
- added joint pinky_23: type revolute, parent d3-1_urdf, child d2-1_urdf, origin xyz=-0.0010000000000001049716 -0.037874999999999880984 -0.00050000000000009411916 rpy=-1.2212476320222462198e-15 4.3296185396076653551e-15 -1.570796326794896336, axis 0 0 1, limit lower=0 upper=1.570796326794896558 effort=1 velocity=20
- added joint pinky_34: type revolute, parent d2-1_urdf, child d1-1_urdf, origin xyz=0.026000000000000078604 2.5413698923060223933e-16 -0.00050000000000020514146 rpy=-2.6352799622801008862e-16 4.944229418462387411e-15 -1.5707963267948958919, axis 0 0 1, limit lower=0 upper=1.570796326794896558 effort=1 velocity=20
- added joint ring_01: type revolute, parent left_forearm_and_palm_assembly, child d4-2_urdf, origin xyz=-0.011784350148794277974 0.19516197601440893328 -0.01051396557923191255 rpy=-3.0545918230670441318 -0.0068123514634775093196 -1.5321205940965847425, axis 0 0 1, limit lower=-0.29670597283903604735 upper=0.29670597283903604735 effort=1 velocity=20
- added joint ring_12: type revolute, parent d4-2_urdf, child d3-2_urdf, origin xyz=-0.015274999999999983036 0.007250000000000039399 -0.0077499999999999522396 rpy=-1.570796326794896558 -1.5707963267948961139 0, axis 0 0 1, limit lower=-0.034906585039886590949 upper=1.570796326794896558 effort=1 velocity=20
- added joint ring_23: type revolute, parent d3-2_urdf, child d2-2_urdf, origin xyz=-0.0010000000000000579172 -0.037875000000000103029 -0.00049999999999996574962 rpy=-6.6268267847551512137e-16 -1.0385351093495972025e-15 -1.570796326794896336, axis 0 0 1, limit lower=0 upper=1.570796326794896558 effort=1 velocity=20
- added joint ring_34: type revolute, parent d2-2_urdf, child d1-2_urdf, origin xyz=0.025999999999999967581 -3.1035287187397564423e-18 -0.00050000000000005768996 rpy=-7.9116884346704368568e-16 -8.8844589975538007006e-17 -1.570796326794961173, axis 0 0 1, limit lower=0 upper=1.570796326794896558 effort=1 velocity=20
- added joint thumb_01: type revolute, parent left_forearm_and_palm_assembly, child t4_urdf, origin xyz=0.014693518066513852616 0.1457335573584342403 -0.026000647022553169396 rpy=1.5707963267948956698 -0.79305228016610029851 -2.9670597283903590302, axis 0 0 1, limit lower=-0.785398163397448279 upper=0.785398163397448279 effort=1 velocity=20
- added joint thumb_12: type revolute, parent t4_urdf, child t3_urdf, origin xyz=-0.016524999999999942513 0.0087500000000000147105 -0.0098249999999999448885 rpy=-1.5707963267948956698 -1.2740903539558086077 1.7268164178027235758e-15, axis 0 0 1, limit lower=0.29670597283903604735 upper=1.570796326794896558 effort=1 velocity=20
- added joint thumb_23: type revolute, parent t3_urdf, child t2_urdf, origin xyz=7.4999999997826805043e-05 -0.04037500000000003586 -0.0015000000000000117406 rpy=6.1081011884469684777e-17 6.564696342128399405e-16 -1.5707963267948970021, axis 0 0 1, limit lower=0 upper=1.570796326794896558 effort=1 velocity=20
- added joint thumb_34: type revolute, parent t2_urdf, child t1_urdf, origin xyz=0.02699999999999996847 5.5511151231257827021e-17 -0.0010000000000000078271 rpy=3.4009006915900816602e-16 1.5792640726178881672e-15 -1.57079632679489678, axis 0 0 1, limit lower=0 upper=1.570796326794896558 effort=1 velocity=20

File: urdf/artus_lite_mk7/right_hand/robot.urdf (robot description, URDF)
Before this commit: robot ArtusLite_RightHand, 22 links, 21 joints
Links:
- removed link r_d1-1_urdf
- removed link r_d1-2_urdf
- removed link r_d1-3_urdf
- removed link r_d1-4_urdf
- removed link r_d2-1_urdf
- removed link r_d2-2_urdf
- removed link r_d2-3_urdf
- removed link r_d2-4_urdf
- removed link r_d3-1_urdf
- removed link r_d3-2_urdf
- removed link r_d3-3_urdf
- removed link r_d3-4_urdf
- removed link r_d4-1_urdf
- removed link r_d4-2_urdf
- removed link r_d4-3_urdf
- removed link r_d4-4_urdf
- removed link r_t1_urdf
- removed link r_t2_urdf
- removed link r_t3_urdf
- removed link r_t4_urdf
- added link d1-1_urdf, mass 0.0096628566425330745387; collision mesh filename=meshes/d1-1_urdf.stl; visual mesh filename=meshes/d1-1_urdf.stl
- added link d1-2_urdf, mass 0.009662856642533072804; collision mesh filename=meshes/d1-2_urdf.stl; visual mesh filename=meshes/d1-2_urdf.stl
- added link d1-3_urdf, mass 0.0096628566425330745387; collision mesh filename=meshes/d1-3_urdf.stl; visual mesh filename=meshes/d1-3_urdf.stl
- added link d1-4_urdf, mass 0.009662856642533072804; collision mesh filename=meshes/d1-4_urdf.stl; visual mesh filename=meshes/d1-4_urdf.stl
- added link d2-1_urdf, mass 0.011864989574403397507; collision mesh filename=meshes/d2-1_urdf.stl; visual mesh filename=meshes/d2-1_urdf.stl
- added link d2-2_urdf, mass 0.011864989574403399242; collision mesh filename=meshes/d2-2_urdf.stl; visual mesh filename=meshes/d2-2_urdf.stl
- added link d2-3_urdf, mass 0.011864989574403397507; collision mesh filename=meshes/d2-3_urdf.stl; visual mesh filename=meshes/d2-3_urdf.stl
- added link d2-4_urdf, mass 0.011864989574403399242; collision mesh filename=meshes/d2-4_urdf.stl; visual mesh filename=meshes/d2-4_urdf.stl
- added link d3-1_urdf, mass 0.022614819883081289931; collision mesh filename=meshes/d3-1_urdf.stl; visual mesh filename=meshes/d3-1_urdf.stl
- added link d3-2_urdf, mass 0.0226148198830812934; collision mesh filename=meshes/d3-2_urdf.stl; visual mesh filename=meshes/d3-2_urdf.stl
- added link d3-3_urdf, mass 0.022614819883081289931; collision mesh filename=meshes/d3-3_urdf.stl; visual mesh filename=meshes/d3-3_urdf.stl
- added link d3-4_urdf, mass 0.022614819883081289931; collision mesh filename=meshes/d3-4_urdf.stl; visual mesh filename=meshes/d3-4_urdf.stl
- added link d4-1_urdf, mass 0.007132231448786834245; collision mesh filename=meshes/d4-1_urdf.stl; visual mesh filename=meshes/d4-1_urdf.stl
- added link d4-2_urdf, mass 0.007132231448786834245; collision mesh filename=meshes/d4-2_urdf.stl; visual mesh filename=meshes/d4-2_urdf.stl
- added link d4-3_urdf, mass 0.0071322314487868333777; collision mesh filename=meshes/d4-3_urdf.stl; visual mesh filename=meshes/d4-3_urdf.stl
- added link d4-4_urdf, mass 0.007132231448786834245; collision mesh filename=meshes/d4-4_urdf.stl; visual mesh filename=meshes/d4-4_urdf.stl
- added link t1_urdf, mass 0.011648615104362203959; collision mesh filename=meshes/t1_urdf.stl; visual mesh filename=meshes/t1_urdf.stl
- added link t2_urdf, mass 0.014650153995995375544; collision mesh filename=meshes/t2_urdf.stl; visual mesh filename=meshes/t2_urdf.stl
- added link t3_urdf, mass 0.030585609045160683933; collision mesh filename=meshes/t3_urdf.stl; visual mesh filename=meshes/t3_urdf.stl
- added link t4_urdf, mass 0.010288104754589431911; collision mesh filename=meshes/t4_urdf.stl; visual mesh filename=meshes/t4_urdf.stl
- link right_forearm_and_palm_assembly: mass 0.35339007201903394062 -> 0.68623229347541214729
Joints:
- removed joint r_index_01
- removed joint r_index_12
- removed joint r_index_23
- removed joint r_index_34
- removed joint r_middle_01
- removed joint r_middle_12
- removed joint r_middle_23
- removed joint r_middle_34
- removed joint r_pinky_01
- removed joint r_pinky_12
- removed joint r_pinky_23
- removed joint r_pinky_34
- removed joint r_ring_01
- removed joint r_ring_12
- removed joint r_ring_23
- removed joint r_ring_34
- removed joint r_thumb_01
- removed joint r_thumb_12
- removed joint r_thumb_23
- removed joint r_thumb_34
- added joint index_01: type revolute, parent right_forearm_and_palm_assembly, child d4-4_urdf, origin xyz=0.03526125935230802616 0.19513802398559065843 0.010513965579232242148 rpy=0.087266462599716959625 5.9001432083974589266e-17 -1.6100662349647696381, axis 0 0 1, limit lower=-0.29670597283903604735 upper=0.29670597283903604735 effort=1 velocity=20
- added joint index_12: type revolute, parent d4-4_urdf, child d3-4_urdf, origin xyz=-0.015274999999999927525 0.0072500000000000168476 -0.0077499999999999912709 rpy=-1.5707963267948941155 -1.570796326794896336 0, axis 0 0 1, limit lower=-0.034906585039886590949 upper=1.570796326794896558 effort=1 velocity=20
- added joint index_23: type revolute, parent d3-4_urdf, child d2-4_urdf, origin xyz=-0.00099999999999992456035 -0.037874999999999880984 -0.00049999999999984084953 rpy=-1.0736478731469521164e-15 -6.4972537115075657867e-15 -1.57079632679489678, axis 0 0 1, limit lower=0 upper=1.570796326794896558 effort=1 velocity=20
- added joint index_34: type revolute, parent d2-4_urdf, child d1-4_urdf, origin xyz=0.025999999999999995337 1.8973538018496327595e-17 -0.00050000000000000044409 rpy=6.9057684691951674976e-15 1.7165371139413334888e-14 -1.5707963267948905628, axis 0 0 1, limit lower=0 upper=1.570796326794896558 effort=1 velocity=20
- added joint middle_01: type revolute, parent right_forearm_and_palm_assembly, child d4-3_urdf, origin xyz=0.01173845611417019541 0.19914999999999996594 0.0080006470225533771884 rpy=-1.3866381960025091427e-17 1.1102487805056423062e-16 -1.5707963267948974462, axis 0 0 1, limit lower=-0.29670597283903604735 upper=0.29670597283903604735 effort=1 velocity=20
- added joint middle_12: type revolute, parent d4-3_urdf, child d3-3_urdf, origin xyz=-0.015274999999999983036 0.0072499999999999821532 -0.0077499999999999617806 rpy=-1.5707963267948941155 -1.5707963267948961139 0, axis 0 0 1, limit lower=-0.034906585039886590949 upper=1.570796326794896558 effort=1 velocity=20
- added joint middle_23: type revolute, parent d3-3_urdf, child d2-3_urdf, origin xyz=-0.0010000000000000451236 -0.037875000000000075273 -0.00049999999999995187183 rpy=1.4009774771081203282e-15 -5.8917067141199026395e-16 -1.5707963267948970021, axis 0 0 1, limit lower=0 upper=1.570796326794896558 effort=1 velocity=20
- added joint middle_34: type revolute, parent d2-3_urdf, child d1-3_urdf, origin xyz=0.02599999999999991207 -1.4755991567527715347e-16 -0.00050000000000009411916 rpy=1.374019371753883429e-15 1.010804088085701642e-15 -1.5707963267948958919, axis 0 0 1, limit lower=0 upper=1.570796326794896558 effort=1 velocity=20
- added joint pinky_01: type revolute, parent right_forearm_and_palm_assembly, child d4-1_urdf, origin xyz=-0.035163937935848779692 0.18909438839224823603 0.014053824767915794672 rpy=-0.17453292519943353067 1.1456913421203554045e-15 -1.4791665410651946289, axis 0 0 1, limit lower=-0.29670597283903604735 upper=0.29670597283903604735 effort=1 velocity=20
- added joint pinky_12: type revolute, parent d4-1_urdf, child d3-1_urdf, origin xyz=-0.015275000000000121814 0.0072500000000001157269 -0.0077499999999997119804 rpy=-1.5707963267948918951 -1.5707963267948952257 0, axis 0 0 1, limit lower=-0.034906585039886590949 upper=1.570796326794896558 effort=1 velocity=20
- added joint pinky_23: type revolute, parent d3-1_urdf, child d2-1_urdf, origin xyz=-0.0010000000000003552054 -0.037875000000000297318 -0.00049999999999856582777 rpy=-2.7917766663472194013e-15 -4.5153227605194488046e-15 -1.5707963267948992225, axis 0 0 1, limit lower=0 upper=1.570796326794896558 effort=1 velocity=20
- added joint pinky_34: type revolute, parent d2-1_urdf, child d1-1_urdf, origin xyz=0.025999999999999967581 -4.7704895589362195096e-18 -0.00049999999999998136213 rpy=5.0133770924262931337e-15 1.4789047887596532477e-15 -1.5707963267948970021, axis 0 0 1, limit lower=0 upper=1.570796326794896558 effort=1 velocity=20
- added joint ring_01: type revolute, parent right_forearm_and_palm_assembly, child d4-2_urdf, origin xyz=-0.011784347123967246762 0.19516197601440882226 0.010513965579232013164 rpy=-0.087000830522749331153 0.0068123514634783575994 -1.5321205940965849646, axis 0 0 1, limit lower=-0.29670597283903604735 upper=0.29670597283903604735 effort=1 velocity=20
- added joint ring_12: type revolute, parent d4-2_urdf, child d3-2_urdf, origin xyz=-0.015275000000000066303 0.0072500000000000116435 -0.0077499999999999045347 rpy=-1.5707963267948992225 -1.5707963267948885644 0, axis 0 0 1, limit lower=-0.034906585039886590949 upper=1.570796326794896558 effort=1 velocity=20
- added joint ring_23: type revolute, parent d3-2_urdf, child d2-2_urdf, origin xyz=-0.0010000000000004540847 -0.037874999999999797717 -0.00050000000000015808709 rpy=4.6419088965683682166e-17 4.5000038854484199404e-15 -1.5707963267948970021, axis 0 0 1, limit lower=0 upper=1.570796326794896558 effort=1 velocity=20
- added joint ring_34: type revolute, parent d2-2_urdf, child d1-2_urdf, origin xyz=0.026000000000000217382 1.0997875787149835602e-17 -0.00050000000000001345452 rpy=4.9184194849935814842e-16 5.9160570651602741219e-16 -1.5707963267948952257, axis 0 0 1, limit lower=0 upper=1.570796326794896558 effort=1 velocity=20
- added joint thumb_01: type revolute, parent right_forearm_and_palm_assembly, child t4_urdf, origin xyz=0.014693521091338347662 0.14573355735843276926 0.026000647022553294296 rpy=1.5707963267948972241 0.79305228016606710284 -2.9670597283903594743, axis 0 0 1, limit lower=-0.785398163397448279 upper=0.785398163397448279 effort=1 velocity=20
- added joint thumb_12: type revolute, parent t4_urdf, child t3_urdf, origin xyz=-0.016524999999999866185 0.0087500000000000511396 -0.0098249999999993342659 rpy=-1.570796326794901443 -1.2740903539558616764 -4.5001425164792760456e-15, axis 0 0 1, limit lower=0.29670597283903604735 upper=1.570796326794896558 effort=1 velocity=20
- added joint thumb_23: type revolute, parent t3_urdf, child t2_urdf, origin xyz=7.4999999999450506216e-05 -0.040374999999997690514 -0.0015000000000003914282 rpy=1.5022520038205650076e-14 2.0353434029585057533e-14 -1.5707963267948945596, axis 0 0 1, limit lower=0 upper=1.570796326794896558 effort=1 velocity=20
- added joint thumb_34: type revolute, parent t2_urdf, child t1_urdf, origin xyz=0.02699999999999996847 -4.1633363423443370266e-17 -0.0010000000000000286438 rpy=2.0108136658001474543e-14 -1.3535182064577502269e-14 -1.57079632679489678, axis 0 0 1, limit lower=0 upper=1.570796326794896558 effort=1 velocity=20
